Commit message: Second commit

File: turtlebot2i_description/robots/kobuki_interbotix_astra.urdf.xacro (robot description, xacro)
@@ -12,6 +12,6 @@
   <sensor_astra parent="base_link"/>
   <sensor_sr300 parent="plate_top_link"/>
-  <phantomx_pincher_arm parent="base_link" color="Red" gripper_color="Red">
+  <!--<phantomx_pincher_arm parent="base_link" color="Red" gripper_color="Red">
     <origin xyz="0.145 0.0 0.124"/>
-  </phantomx_pincher_arm>
+  </phantomx_pincher_arm>-->
 </robot>

File: turtlebot2i_description/robots/kobuki_interbotix_zr300.urdf.xacro (robot description, xacro)
@@ -12,6 +12,6 @@
   <sensor_zr300 parent="base_link"/>
   <sensor_sr300 parent="base_link"/>
-  <phantomx_pincher_arm parent="base_link" color="Red" gripper_color="Red">
+  <!--<phantomx_pincher_arm parent="base_link" color="Red" gripper_color="Red">
     <origin xyz="0.145 0.0 0.124"/>
-  </phantomx_pincher_arm>
+  </phantomx_pincher_arm>-->
 </robot>

File: turtlebot2i_description/urdf/stacks/interbotix.urdf.xacro (robot description, xacro)
@@ -3,4 +3,5 @@
   <!-- TODO: Intertia fields do not contain valid data. Follow tutorial to correct them: http://gazebosim.org/tutorials?tut=inertia -->
   <xacro:include filename="$(find turtlebot2i_description)/urdf/common_properties.urdf.xacro"/>
+  <xacro:include filename="$(find doris_sensors_description)/urdf/hokuyo.urdf.xacro" />
   <!-- Xacro properties -->
   <xacro:property name="PLATE_HEIGHT" value="0.0046"/>
@@ -8,5 +9,5 @@
   <xacro:property name="STANDOFF_100_HEIGHT" value="0.1"/>
   <xacro:property name="STANDOFF_258_HEIGHT" value="0.258"/>
-  <xacro:property name="KOBUKI_TOP_HEIGHT" value="0.0975"/> <!--Measure the floor to the top of the robot base where the standoffs install-->
+  <xacro:property name="KOBUKI_TOP_HEIGHT" value="0.0975"/> <!--Measure the floors to the top of the robot base where the standoffs install-->
   <xacro:property name="BASE_LINK_HEIGHT" value="0.0102"/> <!--TODO: Base link for turtlebot is 10.2mm from floor. Why? -->
   <xacro:property name="STANDOFF_BOTTOM_Z" value="${KOBUKI_TOP_HEIGHT+STANDOFF_50_HEIGHT/2.0-BASE_LINK_HEIGHT}"/>
@@ -327,4 +328,5 @@
     <standoff_258mm parent="${parent}" number="0" x_loc= "0.069" y_loc= "0.130" z_loc="${STANDOFF_FRONT_Z}"/>
     <standoff_258mm parent="${parent}" number="1" x_loc= "0.069" y_loc="-0.130" z_loc="${STANDOFF_FRONT_Z}"/>
+    <xacro:sensor_hokuyo parent="plate_bottom_link" xyz="${0.175 + 0.017 + 0.024 - 0.06} 0 ${0.02 - KOBUKI_TOP_HEIGHT/2}" rpy="3.14 0 0" name="ground"/>
   </xacro:macro>
 </robot>

File: turtlebot2i_description/urdf/turtlebot_library.urdf.xacro (robot description, xacro)
@@ -17,4 +17,4 @@
   <xacro:include filename="$(find turtlebot2i_description)/urdf/sensors/zr300.urdf.xacro"/>
   <!-- Arms -->
-  <xacro:include filename="$(find turtlebot2i_description)/urdf/arms/phantomx_pincher_arm.urdf.xacro"/>
+  <!--<xacro:include filename="$(find turtlebot2i_description)/urdf/arms/phantomx_pincher_arm.urdf.xacro"/>-->
 </robot>

Commit message: feat:posiçao do hokuyo alterada

File: turtlebot2i_description/robots/kobuki_interbotix_astra.urdf.xacro (robot description, xacro)
@@ -12,5 +12,5 @@
   <sensor_astra parent="base_link"/>
   <sensor_sr300 parent="plate_top_link"/>
-  <!--<phantomx_pincher_arm parent="base_link" color="Red" gripper_color="Red">
+  <!--<phantomx_pincher_arm parent="base_footprint" color="Red" gripper_color="Red">
     <origin xyz="0.145 0.0 0.124"/>
   </phantomx_pincher_arm>-->

File: turtlebot2i_description/robots/kobuki_interbotix_zr300.urdf.xacro (robot description, xacro)
@@ -12,6 +12,6 @@
   <sensor_zr300 parent="base_link"/>
   <sensor_sr300 parent="base_link"/>
-  <!--<phantomx_pincher_arm parent="base_link" color="Red" gripper_color="Red">
+  <phantomx_pincher_arm parent="base_link" color="Red" gripper_color="Red">
     <origin xyz="0.145 0.0 0.124"/>
-  </phantomx_pincher_arm>-->
+  </phantomx_pincher_arm>
 </robot>

File: turtlebot2i_description/urdf/arms/phantomx_pincher_arm.urdf.xacro (robot description, xacro)
@@ -3,5 +3,5 @@
 <robot name="phantomx_pincher_arm" xmlns:xacro="http://ros.org/wiki/xacro">
     <!-- We can configure joints velocity limit and lower/upper limits
-          to allow access to different operational areas, e.g. left handed vs. right handed robot -->
+    to allow access to different operational areas, e.g. left handed vs. right handed robot -->
     <xacro:property name="joints_vlimit" value="1.571"/>
     <xacro:property name="pan_llimit" value="-1.74"/>
@@ -14,4 +14,10 @@
     <xacro:property name="wrist_ulimit" value="1.67"/>
     <!-- Included URDF Files -->
-    <xacro:include filename="$(find phantomx_pincher_arm_description)/urdf/phantomx_pincher_arm.xacro" />
+    <xacro:include filename="$(find turtlebot2i_description)/urdf/arms/phantomx_pincher_arm.xacro"/>
+    <!-- As we don't have a base here, add a base_link link as location reference -->
+    <link name="base_footprint"/>
+    <!-- phantomx_pincher_arm macro //joints_vlimit="${joints_vlimit}" pan_llimit="-2.617" pan_ulimit="2.617// -->
+    <phantomx_pincher_arm parent="base_footprint" color="White" gripper_color="White">
+        <origin xyz="0.0 0.00 0.077"/>
+    </phantomx_pincher_arm>
 </robot>

File: turtlebot2i_description/urdf/stacks/interbotix.urdf.xacro (robot description, xacro)
@@ -4,4 +4,5 @@
   <xacro:include filename="$(find turtlebot2i_description)/urdf/common_properties.urdf.xacro"/>
   <xacro:include filename="$(find doris_sensors_description)/urdf/hokuyo.urdf.xacro" />
+  <!--<xacro:include filename="$(find turtlebot2i_description)/urdf/arms/phantomx_pincher_arm.urdf.xacro" />-->
   <!-- Xacro properties -->
   <xacro:property name="PLATE_HEIGHT" value="0.0046"/>
@@ -328,5 +329,8 @@
     <standoff_258mm parent="${parent}" number="0" x_loc= "0.069" y_loc= "0.130" z_loc="${STANDOFF_FRONT_Z}"/>
     <standoff_258mm parent="${parent}" number="1" x_loc= "0.069" y_loc="-0.130" z_loc="${STANDOFF_FRONT_Z}"/>
-    <xacro:sensor_hokuyo parent="plate_bottom_link" xyz="${0.175 + 0.017 + 0.024 - 0.06} 0 ${0.02 - KOBUKI_TOP_HEIGHT/2}" rpy="3.14 0 0" name="ground"/>
+    <xacro:sensor_hokuyo parent="plate_bottom_link" xyz="0.215 0 ${0.002 - KOBUKI_TOP_HEIGHT/1.1}" rpy="3.14 0 0"/>
   </xacro:macro>
+    <!--<xacro:phantomx_pincher_arm  parent="base_footprint">
+		<origin xyz="0 0 0" rpy="0 0 0" />
+    </xacro:phantomx_pincher_arm>-->
 </robot>
