Commit message: tava no robo

File: robots/kobuki_interbotix_d435i.urdf.xacro (robot description, xacro)
@@ -3,15 +3,21 @@
     - Base      : kobuki
     - Stacks    : interbotix
-    - 3d Sensor : zr300
+    - 3d Sensor : d435
     - arm : TODO: supported arms?
 -->
 <robot name="turtlebot" xmlns:xacro="http://ros.org/wiki/xacro">
+  <xacro:include filename="$(find realsense2_description)/urdf/_d435i.urdf.xacro" />
   <xacro:include filename="$(find turtlebot2i_description)/urdf/turtlebot_library.urdf.xacro" />
   <kobuki/>
   <stack_interbotix parent="base_link"/>
-  <sensor_zr300 parent="arm_base_link"/>
-  <!-- <sensor_sr300 parent="arm_base_link"/> -->
-    <!-- <origin xyz="0.15 0.0 0.48" rpy="0.0 0.0 0.0"/>
-  </sensor_sr300> -->
+  <!-- <xacro:kinect_v2 parent="arm_base_link">
+    <origin xyz="-0.10 0.0 0.41" rpy="0.0 0.56 0.0"/>
+  </xacro:kinect_v2>
+   -->
+  <xacro:sensor_d435i parent="arm_base_link">
+    <!-- <origin xyz="-0.10 0 0.42" rpy="0 0.71 0"/> -->
+    <origin xyz="-0.01 0.0 0.29" rpy="0.0 1.27 0.0"/>
+  </xacro:sensor_d435i>
+  <!-- <sensor_sr300 parent="base_link"/> -->
   <phantomx_pincher_arm parent="base_link" color="Red" gripper_color="Red">
     <origin xyz="0.26 0.0 0.112"/>

File: robots/kobuki_interbotix_kinect_v2.urdf copy.xacro (robot description, xacro)
@@ -3,5 +3,5 @@
     - Base      : kobuki
     - Stacks    : interbotix
-    - 3d Sensor : astra
+    - 3d Sensor : kinect v2
     - arm : TODO: supported arms?
 -->
@@ -10,9 +10,9 @@
   <kobuki/>
   <stack_interbotix parent="base_link"/>
-  <xacro:kinect_v2 parent="plate_top_link">
-    <origin xyz="0.105 0.0 0.02" rpy="0.0 0.56 0.0"/>
+  <xacro:kinect_v2 parent="arm_base_link">
+    <origin xyz="-0.10 0.0 0.41" rpy="0.0 0.56 0.0"/>
   </xacro:kinect_v2>
   <phantomx_pincher_arm parent="base_link" color="Red" gripper_color="Red">
-    <origin xyz="0.235 0.0 0.112"/>
+    <origin xyz="0.26 0.0 0.112"/>
   </phantomx_pincher_arm>
 </robot>

File: urdf/sensors/sr300.urdf.xacro (robot description, xacro)
@@ -4,7 +4,7 @@
   <xacro:include filename="$(find turtlebot2i_description)/urdf/turtlebot_properties.urdf.xacro"/>
   <!-- Intel SR300 parameters -->
-  <xacro:property name="sr300_cam_offset_px" value="0.120" />
+  <xacro:property name="sr300_cam_offset_px" value="-0.1" />
   <xacro:property name="sr300_cam_offset_py" value="0.0" />
-  <xacro:property name="sr300_cam_offset_pz" value="0.0023" />
+  <xacro:property name="sr300_cam_offset_pz" value="0.4" />
   <xacro:property name="sr300_cam_rgb_px" value="0.0"/>
   <xacro:property name="sr300_cam_rgb_py" value="0.02403"/>
@@ -57,5 +57,5 @@
     ==  RGB joints & links ==
     -->
-    <joint name="camera_sr300_color_joint" type="fixed">
+    <!-- <joint name="camera_sr300_color_joint" type="fixed">
       <origin xyz="${sr300_cam_rgb_px} ${sr300_cam_rgb_py} ${sr300_cam_rgb_pz}" rpy="0 0 0"/>
       <parent link="camera_sr300"/>
@@ -68,9 +68,9 @@
       <child link="camera_sr300_color_optical_frame" />
     </joint>
-    <link name="camera_sr300_color_optical_frame"/>
+    <link name="camera_sr300_color_optical_frame"/> -->
     <!--
     ==  Depth joints & links ==
     -->
-    <joint name="camera_sr300_depth_joint" type="fixed">
+    <!-- <joint name="camera_sr300_depth_joint" type="fixed">
         <origin xyz="0 0 0" rpy="0 0 0" />
         <parent link="camera_sr300" />
@@ -83,5 +83,5 @@
         <child link="camera_sr300_depth_optical_frame" />
     </joint>
-    <link name="camera_sr300_depth_optical_frame"/>
+    <link name="camera_sr300_depth_optical_frame"/> -->
   	<!-- Simulation sensor -->
     <gazebo reference="camera_sr300">

File: urdf/sensors/zr300.urdf.xacro (robot description, xacro)
@@ -4,7 +4,7 @@
   <xacro:include filename="$(find turtlebot2i_description)/urdf/turtlebot_properties.urdf.xacro"/>
   <!-- Xacro properties -->
-  <xacro:property name="zr300_origin_x" value="-0.050"/>
+  <xacro:property name="zr300_origin_x" value="-0.085"/>
   <xacro:property name="zr300_origin_y" value="0.0"/>
-  <xacro:property name="zr300_origin_z" value="0.25"/>
+  <xacro:property name="zr300_origin_z" value="0.395"/>
   <xacro:property name="zr300_rgb_x" value="0.0"/>
   <xacro:property name="zr300_rgb_y" value="-0.028"/>
@@ -16,5 +16,5 @@
     <joint name="camera_joint" type="fixed">
       <origin xyz="${zr300_origin_x} ${zr300_origin_y} ${zr300_origin_z}"
-              rpy="0 0 0"/>
+              rpy="0 0.78 0"/>
       <parent link="${parent}"/>
       <child link="camera_link"/>

File: urdf/stacks/interbotix.urdf.xacro (robot description, xacro)
@@ -12,12 +12,17 @@
   <xacro:property name="KOBUKI_TOP_HEIGHT" value="0.0975"/> <!--Measure the floors to the top of the robot base where the standoffs install-->
   <xacro:property name="BASE_LINK_HEIGHT" value="0.0102"/> <!--TODO: Base link for turtlebot is 10.2mm from floor. Why? -->
+  <!-- <xacro:property name="STANDOFF_BOTTOM_Z" value="${KOBUKI_TOP_HEIGHT+STANDOFF_50_HEIGHT/2.0-BASE_LINK_HEIGHT}"/> -->
+  <xacro:property name="BASE_PLATE_1" value="${STANDOFF_BOTTOM_Z-0.02-PLATE_HEIGHT/2.0}"/>
+  <xacro:property name="BASE_PLATE_2" value="${STANDOFF_BOTTOM_Z-0.02+PLATE_HEIGHT/2.0}"/>
   <xacro:property name="STANDOFF_BOTTOM_Z" value="${KOBUKI_TOP_HEIGHT+STANDOFF_50_HEIGHT/2.0-BASE_LINK_HEIGHT}"/>
   <xacro:property name="PLATE_BOTTOM_Z" value="${STANDOFF_BOTTOM_Z+STANDOFF_50_HEIGHT/2.0+PLATE_HEIGHT/2.0}"/>
   <xacro:property name="STANDOFF_MIDDLE_Z" value="${PLATE_BOTTOM_Z+PLATE_HEIGHT/2.0+STANDOFF_50_HEIGHT/2.0}"/>
   <xacro:property name="PLATE_MIDDLE_Z" value="${STANDOFF_MIDDLE_Z+STANDOFF_50_HEIGHT/2.0+PLATE_HEIGHT/2.0}"/>
-  <xacro:property name="STANDOFF_UTILITY_BOTTOM_Z" value="${PLATE_MIDDLE_Z+PLATE_HEIGHT/2.0+STANDOFF_50_HEIGHT/2.0}"/>
-  <xacro:property name="PLATE_UTILITY_BOTTOM_Z" value="${STANDOFF_UTILITY_BOTTOM_Z+STANDOFF_50_HEIGHT/2.0+PLATE_HEIGHT/2.0}"/>
-  <xacro:property name="STANDOFF_UTILITY_UPPER_Z" value="${PLATE_UTILITY_BOTTOM_Z+PLATE_HEIGHT/2.0+STANDOFF_100_HEIGHT/2.0}"/>
-  <xacro:property name="PLATE_UTILITY_UPPER_Z" value="${STANDOFF_UTILITY_UPPER_Z+STANDOFF_100_HEIGHT/2.0+PLATE_HEIGHT/2.0}"/>
+  <!-- <xacro:property name="STANDOFF_UTILITY_BOTTOM_Z" value="${PLATE_MIDDLE_Z+PLATE_HEIGHT/2.0+STANDOFF_50_HEIGHT/2.0}"/>
+  <xacro:property name="PLATE_UTILITY_BOTTOM_Z" value="${STANDOFF_UTILITY_BOTTOM_Z+STANDOFF_50_HEIGHT/2.0+PLATE_HEIGHT/2.0}"/> -->
+  <xacro:property name="STANDOFF_UTILITY_Z" value="${PLATE_BOTTOM_Z+PLATE_HEIGHT/2+STANDOFF_50_HEIGHT}"/>
+  <xacro:property name="PLATE_UTILITY_Z" value="${STANDOFF_UTILITY_Z+STANDOFF_50_HEIGHT+PLATE_HEIGHT/2}"/>
+  <!-- <xacro:property name="STANDOFF_UTILITY_UPPER_Z" value="${PLATE_UTILITY_BOTTOM_Z+PLATE_HEIGHT/2.0+STANDOFF_100_HEIGHT/2.0}"/>
+  <xacro:property name="PLATE_UTILITY_UPPER_Z" value="${STANDOFF_UTILITY_UPPER_Z+STANDOFF_100_HEIGHT/2.0+PLATE_HEIGHT/2.0}"/> -->
   <xacro:property name="STANDOFF_TOP_Z" value="${PLATE_UTILITY_UPPER_Z+PLATE_HEIGHT/2.0+STANDOFF_100_HEIGHT/2.0}"/>
   <xacro:property name="PLATE_TOP_Z" value="${STANDOFF_TOP_Z+STANDOFF_100_HEIGHT/2.0+PLATE_HEIGHT/2.0}"/>
@@ -26,4 +31,9 @@
     <material name="pink">
       <color rgba="0.8 0.0 0.4 1"/>
+    </material>
+  </xacro:property>
+    <xacro:property name="material_black">
+    <material name="black">
+      <color rgba="0.200 0.200 0.200 1"/>
     </material>
   </xacro:property>
@@ -47,5 +57,5 @@
           <mesh filename="package://turtlebot2i_description/meshes/stacks/interbotix/standoff_50mm.stl"/>
         </geometry>
-        <xacro:insert_block name="material_pink"/>
+        <xacro:insert_block name="material_black"/>
       </visual>
       <collision>
@@ -81,5 +91,5 @@
           <mesh filename="package://turtlebot2i_description/meshes/stacks/interbotix/standoff_100mm.stl"/>
         </geometry>
-        <xacro:insert_block name="material_pink"/>
+        <xacro:insert_block name="material_black"/>
       </visual>
       <collision>
@@ -115,5 +125,5 @@
           <mesh filename="package://turtlebot2i_description/meshes/stacks/interbotix/standoff_258mm.stl"/>
         </geometry>
-        <xacro:insert_block name="material_pink"/>
+        <xacro:insert_block name="material_black"/>
       </visual>
       <collision>
@@ -143,16 +153,16 @@
   -->
   <xacro:macro name="stack_interbotix" params="parent">
-    <standoff_50mm parent="${parent}" number="0" x_loc= "0.120" y_loc= "0.082" z_loc="${STANDOFF_BOTTOM_Z}"/>
+    <!-- <standoff_50mm parent="${parent}" number="0" x_loc= "0.120" y_loc= "0.082" z_loc="${STANDOFF_BOTTOM_Z}"/> -->
     <standoff_50mm parent="${parent}" number="1" x_loc= "0.055" y_loc= "0.120" z_loc="${STANDOFF_BOTTOM_Z}"/>
     <standoff_50mm parent="${parent}" number="2" x_loc="-0.055" y_loc= "0.120" z_loc="${STANDOFF_BOTTOM_Z}"/>
-    <standoff_50mm parent="${parent}" number="3" x_loc= "0.120" y_loc="-0.082" z_loc="${STANDOFF_BOTTOM_Z}"/>
-    <standoff_50mm parent="${parent}" number="4" x_loc= "0.055" y_loc="-0.120" z_loc="${STANDOFF_BOTTOM_Z}"/>
-    <standoff_50mm parent="${parent}" number="5" x_loc="-0.055" y_loc="-0.120" z_loc="${STANDOFF_BOTTOM_Z}"/>
-    <joint name="plate_bottom_joint" type="fixed">
-      <origin xyz="0.0 0.0 ${PLATE_BOTTOM_Z}" rpy="0 0 0"/>
-      <parent link="${parent}"/>
-      <child link="plate_bottom_link"/>
-    </joint>
-    <link name="plate_bottom_link">
+    <!-- <standoff_50mm parent="${parent}" number="3" x_loc= "0.120" y_loc="-0.082" z_loc="${STANDOFF_BOTTOM_Z}"/> -->
+    <standoff_50mm parent="${parent}" number="3" x_loc= "0.055" y_loc="-0.120" z_loc="${STANDOFF_BOTTOM_Z}"/>
+    <standoff_50mm parent="${parent}" number="4" x_loc="-0.055" y_loc="-0.120" z_loc="${STANDOFF_BOTTOM_Z}"/>
+    <joint name="base_plate_joint" type="fixed">
+      <origin xyz="0.11 0.0 ${BASE_PLATE_1}" rpy="0 0 0"/>
+      <parent link="${parent}"/>
+      <child link="base_plate_link"/>
+    </joint>
+    <link name="base_plate_link">
       <visual>
         <origin xyz="0 0 0" rpy="0 0 0"/>
@@ -176,4 +186,36 @@
       </inertial>
     </link>
+    <gazebo reference="base_plate_link">
+      <material>Gazebo/Black</material>
+      <!-- <selfCollide>true</selfCollide> -->
+      <gravity>true</gravity>
+    </gazebo>
+    <joint name="plate_bottom_joint" type="fixed">
+      <origin xyz="0.11 0.0 ${BASE_PLATE_2}" rpy="0 0 0"/>
+      <parent link="${parent}"/>
+      <child link="plate_bottom_link"/>
+    </joint>
+    <link name="plate_bottom_link">
+      <visual>
+        <origin xyz="0 0 0" rpy="0 0 0"/>
+        <geometry>
+          <mesh filename="package://turtlebot2i_description/meshes/stacks/interbotix/TurtleBot2i_BottomPlate.stl"/>
+        </geometry>
+        <xacro:insert_block name="material_near_black"/>
+      </visual>
+      <collision>
+        <origin xyz="0 0 0" rpy="0 0 0"/>
+        <geometry>
+          <cylinder length="0.006" radius="0.170"/>
+        </geometry>
+      </collision>
+      <inertial>
+        <mass value="0.311" />
+        <origin xyz="0 0 0" />
+        <inertia ixx="0.003328" ixy="0.0" ixz="0.0"
+                 iyy="0.003328" iyz="0.0"
+                 izz="0.006656" />
+      </inertial>
+    </link>
     <gazebo reference="plate_bottom_link">
       <material>Gazebo/Black</material>
@@ -181,12 +223,12 @@
       <gravity>true</gravity>
     </gazebo>
-    <standoff_50mm parent="${parent}" number="6" x_loc= "0.069" y_loc= "0.130" z_loc="${STANDOFF_MIDDLE_Z}"/>
+    <!-- <standoff_50mm parent="${parent}" number="6" x_loc= "0.069" y_loc= "0.130" z_loc="${STANDOFF_MIDDLE_Z}"/>
     <standoff_50mm parent="${parent}" number="7" x_loc= "0.069" y_loc="-0.130" z_loc="${STANDOFF_MIDDLE_Z}"/>
     <standoff_50mm parent="${parent}" number="8" x_loc= "-0.001" y_loc= "0.162" z_loc="${STANDOFF_MIDDLE_Z}"/>
     <standoff_50mm parent="${parent}" number="9" x_loc= "-0.001" y_loc="-0.162" z_loc="${STANDOFF_MIDDLE_Z}"/>
     <standoff_50mm parent="${parent}" number="10" x_loc="-0.104" y_loc= "0.098" z_loc="${STANDOFF_MIDDLE_Z}"/>
-    <standoff_50mm parent="${parent}" number="11" x_loc="-0.104" y_loc="-0.098" z_loc="${STANDOFF_MIDDLE_Z}"/>
+    <standoff_50mm parent="${parent}" number="11" x_loc="-0.104" y_loc="-0.098" z_loc="${STANDOFF_MIDDLE_Z}"/> -->
     <joint name="plate_middle_joint" type="fixed">
-      <origin xyz="0.0 0.0 ${PLATE_MIDDLE_Z}" rpy="0 0 0"/>
+      <origin xyz="0.0 0.0 ${PLATE_BOTTOM_Z}" rpy="0 0 0"/>
       <parent link="${parent}"/>
       <child link="plate_middle_link"/>
@@ -219,14 +261,14 @@
       <gravity>true</gravity>
     </gazebo>
-    <standoff_100mm parent="${parent}" number="6" x_loc= "-0.001" y_loc= "0.162" z_loc="${STANDOFF_UTILITY_BOTTOM_Z}"/>
-    <standoff_100mm parent="${parent}" number="7" x_loc= "-0.001" y_loc="-0.162" z_loc="${STANDOFF_UTILITY_BOTTOM_Z}"/>
-    <standoff_100mm parent="${parent}" number="8" x_loc="-0.104" y_loc= "0.098" z_loc="${STANDOFF_UTILITY_BOTTOM_Z}"/>
-    <standoff_100mm parent="${parent}" number="9" x_loc="-0.104" y_loc="-0.098" z_loc="${STANDOFF_UTILITY_BOTTOM_Z}"/>
-    <joint name="plate_utility_lower" type="fixed">
-      <origin xyz="0.0 0.0 ${PLATE_UTILITY_BOTTOM_Z}" rpy="0 0 0"/>
-      <parent link="${parent}"/>
-      <child link="plate_utility_lower_link"/>
-    </joint>
-    <link name="plate_utility_lower_link">
+    <standoff_100mm parent="${parent}" number="6" x_loc= "-0.001" y_loc= "0.162" z_loc="${STANDOFF_UTILITY_Z}"/>
+    <standoff_100mm parent="${parent}" number="7" x_loc= "-0.001" y_loc="-0.162" z_loc="${STANDOFF_UTILITY_Z}"/>
+    <standoff_100mm parent="${parent}" number="8" x_loc="-0.104" y_loc= "0.098" z_loc="${STANDOFF_UTILITY_Z}"/>
+    <standoff_100mm parent="${parent}" number="9" x_loc="-0.104" y_loc="-0.098" z_loc="${STANDOFF_UTILITY_Z}"/>
+    <joint name="plate_utility" type="fixed">
+      <origin xyz="0.0 0.0 ${PLATE_UTILITY_Z}" rpy="0 0 0"/>
+      <parent link="${parent}"/>
+      <child link="plate_utility_link"/>
+    </joint>
+    <link name="plate_utility_link">
       <visual>
         <origin xyz="0 0 0" rpy="0 0 0"/>
@@ -250,84 +292,12 @@
       </inertial>
     </link>
-    <gazebo reference="plate_utility_lower_link">
-      <material>Gazebo/Black</material>
-      <!-- <selfCollide>true</selfCollide> -->
-      <gravity>true</gravity>
-    </gazebo>
-    <standoff_100mm parent="${parent}" number="0" x_loc= "-0.001" y_loc= "0.162" z_loc="${STANDOFF_UTILITY_UPPER_Z}"/>
-    <standoff_100mm parent="${parent}" number="1" x_loc= "-0.001" y_loc="-0.162" z_loc="${STANDOFF_UTILITY_UPPER_Z}"/>
-    <standoff_100mm parent="${parent}" number="2" x_loc="-0.104" y_loc= "0.098" z_loc="${STANDOFF_UTILITY_UPPER_Z}"/>
-    <standoff_100mm parent="${parent}" number="3" x_loc="-0.104" y_loc="-0.098" z_loc="${STANDOFF_UTILITY_UPPER_Z}"/>
-    <joint name="plate_utility_upper" type="fixed">
-      <origin xyz="0.0 0.0 ${PLATE_UTILITY_UPPER_Z}" rpy="0 0 0"/>
-      <parent link="${parent}"/>
-      <child link="plate_utility_upper_link"/>
-    </joint>
-    <link name="plate_utility_upper_link">
-      <visual>
-        <origin xyz="0 0 0" rpy="0 0 0"/>
-        <geometry>
-          <mesh filename="package://turtlebot2i_description/meshes/stacks/interbotix/TurtleBot2i_UtilityPlate.stl"/>
-        </geometry>
-        <xacro:insert_block name="material_near_black"/>
-      </visual>
-      <collision>
-        <origin xyz="0.0 0.0 0.0" rpy="0 0 0"/>
-        <geometry>
-          <mesh filename="package://turtlebot2i_description/meshes/stacks/interbotix/TurtleBot2i_UtilityPlate.stl"/>
-        </geometry>
-      </collision>
-      <inertial>
-        <mass value="0.153" />
-        <origin xyz="0 0 0" />
-        <inertia ixx="0.003328" ixy="0.0" ixz="0.0"
-                 iyy="0.003328" iyz="0.0"
-                 izz="0.006656" />
-      </inertial>
-    </link>
-    <gazebo reference="plate_utility_upper_link">
-      <material>Gazebo/Black</material>
-      <!-- <selfCollide>true</selfCollide> -->
-      <gravity>true</gravity>
-    </gazebo>
-    <standoff_100mm parent="${parent}" number="10" x_loc= "-0.001" y_loc= "0.162" z_loc="${STANDOFF_TOP_Z}"/>
-    <standoff_100mm parent="${parent}" number="11" x_loc= "-0.001" y_loc="-0.162" z_loc="${STANDOFF_TOP_Z}"/>
-    <standoff_100mm parent="${parent}" number="12" x_loc="-0.104" y_loc= "0.098" z_loc="${STANDOFF_TOP_Z}"/>
-    <standoff_100mm parent="${parent}" number="13" x_loc="-0.104" y_loc="-0.098" z_loc="${STANDOFF_TOP_Z}"/>
-    <joint name="plate_top_joint" type="fixed">
-      <origin xyz="0.0 0.0 ${PLATE_TOP_Z}" rpy="0 0 0"/>
-      <parent link="${parent}"/>
-      <child link="plate_top_link"/>
-    </joint>
-    <link name="plate_top_link">
-      <visual>
-        <origin xyz="0 0 0" rpy="0 0 0"/>
-        <geometry>
-          <mesh filename="package://turtlebot2i_description/meshes/stacks/interbotix/TurtleBot2i_TopPlate.stl" scale="0.001 0.001 0.001"/>
-        </geometry>
-        <xacro:insert_block name="material_near_black"/>
-      </visual>
-      <collision>
-        <origin xyz="0 0 0" rpy="0 0 0"/>
-        <geometry>
-          <mesh filename="package://turtlebot2i_description/meshes/stacks/interbotix/TurtleBot2i_TopPlate.stl" scale="0.001 0.001 0.001"/>
-        </geometry>
-      </collision>
-      <inertial>
-        <mass value="0.377"/>
-        <origin xyz="0 0 0"/>
-        <inertia ixx="0.003328" ixy="0.0" ixz="0.0"
-                 iyy="0.003328" iyz="0.0"
-                 izz="0.006656" />
-      </inertial>
-    </link>
-    <gazebo reference="plate_top_link">
-      <material>Gazebo/Black</material>
-      <!-- <selfCollide>true</selfCollide> -->
-      <gravity>true</gravity>
-    </gazebo>
-    <standoff_258mm parent="${parent}" number="0" x_loc= "0.069" y_loc= "0.130" z_loc="${STANDOFF_FRONT_Z}"/>
-    <standoff_258mm parent="${parent}" number="1" x_loc= "0.069" y_loc="-0.130" z_loc="${STANDOFF_FRONT_Z}"/>
-    <xacro:sensor_hokuyo parent="plate_bottom_link" xyz="0.215 0 ${0.002 - KOBUKI_TOP_HEIGHT/1.1}" rpy="3.14 0 0"/>
+    <gazebo reference="plate_utility_link">
+      <material>Gazebo/Black</material>
+      <!-- <selfCollide>true</selfCollide> -->
+      <gravity>true</gravity>
+    </gazebo>
+    <!-- <standoff_258mm parent="${parent}" number="0" x_loc= "0.069" y_loc= "0.130" z_loc="${STANDOFF_FRONT_Z}"/>
+    <standoff_258mm parent="${parent}" number="1" x_loc= "0.069" y_loc="-0.130" z_loc="${STANDOFF_FRONT_Z}"/> -->
+    <xacro:sensor_hokuyo parent="plate_bottom_link" xyz="0.1 0 -0.035" rpy="3.14 0 0"/>
     </xacro:macro>
     <!--<xacro:kinect_v2 parent="plate_top_link">

File: urdf/turtlebot_library.urdf.xacro (robot description, xacro)
@@ -13,8 +13,8 @@
   <xacro:include filename="$(find turtlebot2i_description)/urdf/stacks/interbotix.urdf.xacro"/>
   <!-- 3D Sensors -->
-  <!--<xacro:include filename="$(find turtlebot2i_description)/urdf/sensors/astra.urdf.xacro"/>-->
-  <!--<xacro:include filename="$(find turtlebot2i_description)/urdf/sensors/sr300.urdf.xacro"/>-->
-  <!--<xacro:include filename="$(find turtlebot2i_description)/urdf/sensors/zr300.urdf.xacro"/>-->
-  <xacro:include filename="$(find kinect_v2)/urdf/kinect_v2.urdf.xacro"/>
+  <xacro:include filename="$(find turtlebot2i_description)/urdf/sensors/astra.urdf.xacro"/>
+  <xacro:include filename="$(find turtlebot2i_description)/urdf/sensors/sr300.urdf.xacro"/>
+  <xacro:include filename="$(find turtlebot2i_description)/urdf/sensors/zr300.urdf.xacro"/>
+  <!--<xacro:include filename="$(find kinect_v2)/urdf/kinect_v2.urdf.xacro"/>-->
   <!-- Arms -->
   <xacro:include filename="$(find turtlebot2i_description)/urdf/arms/phantomx_pincher_arm.urdf.xacro"/>

Commit message: added realsense

File: robots/kobuki_interbotix_d435i.urdf.xacro (robot description, xacro)
@@ -16,6 +16,6 @@
    -->
   <xacro:sensor_d435i parent="arm_base_link">
-    <!-- <origin xyz="-0.10 0 0.42" rpy="0 0.71 0"/> -->
-    <origin xyz="-0.01 0.0 0.29" rpy="0.0 1.27 0.0"/>
+    <!-- <origin xyz="-0.10 0 0.42" rpy="0 0.61 0"/> -->
+    <origin xyz="-0.06 0.0 0.30" rpy="0.0 0.61 0.0"/>
   </xacro:sensor_d435i>
   <!-- <sensor_sr300 parent="base_link"/> -->

Commit message: :recycle: change robot urdf to RoboCup

File: robots/kobuki_interbotix_d435i.urdf.xacro (robot description, xacro)
@@ -14,10 +14,8 @@
     <origin xyz="-0.10 0.0 0.41" rpy="0.0 0.56 0.0"/>
   </xacro:kinect_v2>
-   -->
+  -->
   <xacro:sensor_d435i parent="arm_base_link">
-    <!-- <origin xyz="-0.10 0 0.42" rpy="0 0.61 0"/> -->
-    <origin xyz="-0.06 0.0 0.30" rpy="0.0 0.61 0.0"/>
+    <origin xyz="-0.025  0.0 0.305" rpy="0.0 0.707 0.0"/>
   </xacro:sensor_d435i>
-  <!-- <sensor_sr300 parent="base_link"/> -->
   <phantomx_pincher_arm parent="base_link" color="Red" gripper_color="Red">
     <origin xyz="0.26 0.0 0.112"/>

File: urdf/arms/phantomx_pincher_arm.urdf.xacro (robot description, xacro)
@@ -5,6 +5,6 @@
     to allow access to different operational areas, e.g. left handed vs. right handed robot -->
     <xacro:property name="joints_vlimit" value="1.571"/>
-    <xacro:property name="pan_llimit" value="-1.74"/>
-    <xacro:property name="pan_ulimit" value="1.74"/>
+    <xacro:property name="pan_llimit" value="-3.66"/>
+    <xacro:property name="pan_ulimit" value="3.66"/>
     <xacro:property name="shoulder_llimit" value="-1.98"/>
     <xacro:property name="shoulder_ulimit" value="1.88"/>

Commit message: :wrench: change arm limits  and camera angle

File: robots/kobuki_interbotix_d435i.urdf.xacro (robot description, xacro)
@@ -17,5 +17,5 @@
   <xacro:sensor_d435i parent="arm_base_link">
     <!-- <origin xyz="-0.10 0 0.42" rpy="0 0.61 0"/> -->
-    <origin xyz="-0.06 0.0 0.30" rpy="0.0 0.61 0.0"/>
+    <origin xyz="-0.06 0.0 0.30" rpy="0.0 0.8 0.0"/>
   </xacro:sensor_d435i>
   <!-- <sensor_sr300 parent="base_link"/> -->

File: urdf/arms/phantomx_pincher_arm.urdf.xacro (robot description, xacro)
@@ -4,13 +4,13 @@
     <!-- We can configure joints velocity limit and lower/upper limits
     to allow access to different operational areas, e.g. left handed vs. right handed robot -->
-    <xacro:property name="joints_vlimit" value="1.571"/>
-    <xacro:property name="pan_llimit" value="-1.74"/>
-    <xacro:property name="pan_ulimit" value="1.74"/>
+    <xacro:property name="joints_vlimit" value="2.09"/>
+    <xacro:property name="pan_llimit" value="-2.74"/>
+    <xacro:property name="pan_ulimit" value="2.74"/>
     <xacro:property name="shoulder_llimit" value="-1.98"/>
     <xacro:property name="shoulder_ulimit" value="1.88"/>
     <xacro:property name="elbow_llimit" value="-1.58"/>
-    <xacro:property name="elbow_ulimit" value="0.59"/>
-    <xacro:property name="wrist_llimit" value="-1.79"/>
-    <xacro:property name="wrist_ulimit" value="1.67"/>
+    <xacro:property name="elbow_ulimit" value="0.85"/>
+    <xacro:property name="wrist_llimit" value="-2"/>
+    <xacro:property name="wrist_ulimit" value="2"/>
     <!-- Included URDF Files -->
     <xacro:include filename="$(find phantomx_pincher_arm_description)/urdf/phantomx_pincher_arm.xacro"/>
